Commit message: update

File: robot_navigation/urdf/jackal.urdf (robot description, URDF)
Before this commit: robot jackal, 2 links, 1 joints
Links:
- removed link chassis_link
- added link front_caster_link; visual sphere radius=0.0165
- added link left_motor; visual cylinder length=0.08 radius=0.02
- added link left_wheel_link; visual cylinder length=0.017 radius=0.033
- link base_link: geometry visual box size=0.03 0.02 0.005
Joints:
- removed joint chassis_link_joint
- added joint base_left_motor_joint: type fixed, parent base_link, child left_motor, origin xyz=-0.055 0.075 0 rpy=0 0 0
- added joint front_caster_joint: type fixed, parent base_link, child front_caster_link, origin xyz=0.1135 0 -0.0165 rpy=0 0 0
- added joint left_wheel_joint: type continuous, parent left_motor, child left_wheel_link, origin xyz=0 0.0485 0 rpy=0 0 0, axis 0 1 0
