Commit message: update

File: robot_navigation/urdf/_d435.urdf.xacro (robot description, xacro)
@@ -30,16 +30,16 @@
     </material>
     <!-- camera body, with origin at bottom screw mount -->
-    <joint name="camera_joint" type="fixed">
+    <joint name="d400_joint" type="fixed">
       <xacro:insert_block name="origin" />
       <parent link="${parent}"/>
-      <child link="camera_bottom_screw_frame" />
+      <child link="d400_bottom_screw_frame" />
     </joint>
-    <link name="camera_bottom_screw_frame"/>
-    <joint name="camera_link_joint" type="fixed">
+    <link name="d400_bottom_screw_frame"/>
+    <joint name="d400_link_joint" type="fixed">
       <origin xyz="0 ${d435_cam_depth_py} ${d435_cam_depth_pz}" rpy="0 0 0"/>
-      <parent link="camera_bottom_screw_frame"/>
-      <child link="camera_link" />
+      <parent link="d400_bottom_screw_frame"/>
+      <child link="d400_link" />
     </joint>
-    <link name="camera_link">
+    <link name="d400_link">
       <visual>
       <origin xyz="${d435_cam_mount_from_center_offset} ${-d435_cam_depth_py} 0" rpy="${M_PI/2} 0 ${M_PI/2}"/>
@@ -65,55 +65,55 @@
     </link>
     <!-- camera depth joints and links -->
-    <joint name="camera_depth_joint" type="fixed">
+    <joint name="d400_depth_joint" type="fixed">
       <origin xyz="0 0 0" rpy="0 0 0"/>
-      <parent link="camera_link"/>
-      <child link="camera_depth_frame" />
+      <parent link="d400_link"/>
+      <child link="d400_depth_frame" />
     </joint>
-    <link name="camera_depth_frame"/>
-    <joint name="camera_depth_optical_joint" type="fixed">
+    <link name="d400_depth_frame"/>
+    <joint name="d400_depth_optical_joint" type="fixed">
       <origin xyz="0 0 0" rpy="${-M_PI/2} 0 ${-M_PI/2}" />
-      <parent link="camera_depth_frame" />
-      <child link="camera_depth_optical_frame" />
+      <parent link="d400_depth_frame" />
+      <child link="d400_depth_optical_frame" />
     </joint>
-    <link name="camera_depth_optical_frame"/>
+    <link name="d400_depth_optical_frame"/>
     <!-- camera left IR joints and links -->
-    <joint name="camera_left_ir_joint" type="fixed">
+    <joint name="d400_left_ir_joint" type="fixed">
       <origin xyz="0 ${d435_cam_depth_to_left_ir_offset} 0" rpy="0 0 0" />
-      <parent link="camera_depth_frame" />
-      <child link="camera_left_ir_frame" />
+      <parent link="d400_depth_frame" />
+      <child link="d400_left_ir_frame" />
     </joint>
-    <link name="camera_left_ir_frame"/>
-    <joint name="camera_left_ir_optical_joint" type="fixed">
+    <link name="d400_left_ir_frame"/>
+    <joint name="d400_left_ir_optical_joint" type="fixed">
       <origin xyz="0 0 0" rpy="${-M_PI/2} 0 ${-M_PI/2}" />
-      <parent link="camera_left_ir_frame" />
-      <child link="camera_left_ir_optical_frame" />
+      <parent link="d400_left_ir_frame" />
+      <child link="d400_left_ir_optical_frame" />
     </joint>
-    <link name="camera_left_ir_optical_frame"/>
+    <link name="d400_left_ir_optical_frame"/>
     <!-- camera right IR joints and links -->
-    <joint name="camera_right_ir_joint" type="fixed">
+    <joint name="d400_right_ir_joint" type="fixed">
       <origin xyz="0 ${d435_cam_depth_to_right_ir_offset} 0" rpy="0 0 0" />
-      <parent link="camera_depth_frame" />
-      <child link="camera_right_ir_frame" />
+      <parent link="d400_depth_frame" />
+      <child link="d400_right_ir_frame" />
     </joint>
-    <link name="camera_right_ir_frame"/>
-    <joint name="camera_right_ir_optical_joint" type="fixed">
+    <link name="d400_right_ir_frame"/>
+    <joint name="d400_right_ir_optical_joint" type="fixed">
       <origin xyz="0 0 0" rpy="${-M_PI/2} 0 ${-M_PI/2}" />
-      <parent link="camera_right_ir_frame" />
-      <child link="camera_right_ir_optical_frame" />
+      <parent link="d400_right_ir_frame" />
+      <child link="d400_right_ir_optical_frame" />
     </joint>
-    <link name="camera_right_ir_optical_frame"/>
+    <link name="d400_right_ir_optical_frame"/>
     <!-- camera color joints and links -->
-    <joint name="camera_color_joint" type="fixed">
+    <joint name="d400_color_joint" type="fixed">
       <origin xyz="0 ${d435_cam_depth_to_color_offset} 0" rpy="0 0 0" />
-      <parent link="camera_depth_frame" />
-      <child link="camera_color_frame" />
+      <parent link="d400_depth_frame" />
+      <child link="d400_color_frame" />
     </joint>
-    <link name="camera_color_frame"/>
-    <joint name="camera_color_optical_joint" type="fixed">
+    <link name="d400_color_frame"/>
+    <joint name="d400_color_optical_joint" type="fixed">
       <origin xyz="0 0 0" rpy="${-M_PI/2} 0 ${-M_PI/2}" />
-      <parent link="camera_color_frame" />
-      <child link="camera_color_optical_frame" />
+      <parent link="d400_color_frame" />
+      <child link="d400_color_optical_frame" />
     </joint>
-    <link name="camera_color_optical_frame"/>
+    <link name="d400_color_optical_frame"/>
   </xacro:macro>
 </robot>

File: robot_navigation/urdf/jackal.urdf.xacro (robot description, xacro)
@@ -17,4 +17,5 @@
   <material name="yellow"><color rgba="0.8 0.8 0.0 1.0" /></material>
   <material name="black"><color rgba="0.15 0.15 0.15 1.0" /></material>
+ <!--
   <xacro:macro name="wheel" params="prefix *joint_pose">
     <link name="${prefix}_wheel_link">
@@ -56,6 +57,4 @@
       <axis xyz="0 1 0" />
     </joint>
-    <!-- In reality, Jackal has only two motors, one per side. However, it's more
-         straightforward for Gazebo to simulate as if there's an actuator per wheel. -->
     <transmission name="${prefix}_wheel_trans">
       <type>transmission_interface/SimpleTransmission</type>
@@ -80,4 +79,5 @@
     <origin xyz="${-wheelbase/2} ${-track/2} ${wheel_vertical_offset}" rpy="0 0 0" />
   </xacro:wheel>
+-->
   <link name="base_link"></link>
   <joint name="base_link_joint" type="fixed">
@@ -217,8 +217,14 @@
     <origin xyz="${mount_spacing} 0 0" />
   </joint>
+  <link name="front_laser"></link>
+  <joint name="front_laser_joint" type="fixed">
+    <parent link="front_mount" />
+    <child link="front_laser" />
+    <origin xyz="0 0 0.05" />
+  </joint>
   <xacro:include filename="$(find robot_navigation)/urdf/accessories.urdf.xacro" />
   <xacro:include filename="$(find robot_navigation)/urdf/_d435.urdf.xacro" />
   <sensor_d435 parent="mid_mount">
-    <origin xyz="0 0 0" rpy="0 0 0"/>
+    <origin xyz="-0.02 0 0.2" rpy="0 0 0"/>
   </sensor_d435>
 </robot>
