Commit message: update

File: robot_navigation/urdf/hokuyo_ust10.urdf.xacro (robot description, xacro)
@@ -8,9 +8,9 @@
           <mesh filename="package://jackal_description/meshes/hokuyo_ust10.stl" />
         </geometry>
-        <material name="dark_grey" />
+        <material name="light_grey" />
       </visual>
     </link>
     <joint name="${prefix}_laser_mount_joint" type="fixed">
-      <origin xyz="0 0 0" rpy="0 0 0" />
+      <origin xyz="0.04 0.0 0.01" rpy="0 0 0" />
       <parent link="${parent_link}" />
       <child link="${prefix}_laser_mount" />

File: robot_navigation/urdf/jackal_desktop.urdf.xacro (robot description, xacro)
@@ -273,5 +273,5 @@
   <xacro:include filename="$(find robot_navigation)/urdf/_d435.urdf.xacro" />
   <sensor_d435 parent="mid_mount">
-    <origin xyz="-0.02 0 0.2" rpy="0 0 0"/>
+    <origin xyz="0.0 0.0 0.3" rpy="0 0 0"/>
   </sensor_d435>
   <xacro:include filename="$(find robot_navigation)/urdf/hokuyo_ust10.urdf.xacro" />
